File: _autosave-Custom Keyboard STM32.kicad_pcb (KiCad board)
At the start: 2 copper layers, 10.1 x 6.4 mm, 217 parts, among them Q1 2N7002, U1 XC6206P332MR, U2 IS31FL3733-TQ, U3 IS31FL3733-TQ, U4 STM32F303CBT6, U5 SRV05-4

Commit message: 1
Parts:
- moved D1 12.7 mm to (45.3, 43.9), turned to 180 degrees
Changed lines of the file:
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@@
       (effects (font (size 0.5 0.5) (thickness 0.08)))
     )
-    (fp_line (start -0.227064 0.735) (end 0.227064 0.735) (layer "F.SilkS") (width 0.12))
     (fp_line (start -0.227064 -0.735) (end 0.227064 -0.735) (layer "F.SilkS") (width 0.12))
+    (fp_line (start -0.227064 0.735) (end 0.227064 0.735) (layer "F.SilkS") (width 0.12))
     (fp_line (start -1.68 0.95) (end -1.68 -0.95) (layer "F.CrtYd") (width 0.05))
     (fp_line (start 1.68 0.95) (end -1.68 0.95) (layer "F.CrtYd") (width 0.05))
@@
       (effects (font (size 0.4 0.4) (thickness 0.06)))
     )
-    (fp_line (start 0 1.56) (end 0.8 1.56) (layer "F.SilkS") (width 0.12))
     (fp_line (start -2.1 -1.56) (end 0.8 -1.56) (layer "F.SilkS") (width 0.12))
     (fp_line (start -2.1 -0.95) (end -2.1 -1.56) (layer "F.SilkS") (width 0.12))
     (fp_line (start 0 1.56) (end -0.8 1.56) (layer "F.SilkS") (width 0.12))
+    (fp_line (start 0 1.56) (end 0.8 1.56) (layer "F.SilkS") (width 0.12))
     (fp_line (start -2.05 -1.7) (end -2.05 1.7) (layer "F.CrtYd") (width 0.05))
     (fp_line (start -2.05 1.7) (end 2.05 1.7) (layer "F.CrtYd") (width 0.05))
@@
     (fp_line (start 1.68 0.95) (end -1.68 0.95) (layer "F.CrtYd") (width 0.05))
     (fp_line (start -1.68 -0.95) (end 1.68 -0.95) (layer "F.CrtYd") (width 0.05))
-    (fp_line (start -1 -0.625) (end 1 -0.625) (layer "F.Fab") (width 0.1))
     (fp_line (start -1 0.625) (end -1 -0.625) (layer "F.Fab") (width 0.1))
+    (fp_line (start -1 -0.625) (end 1 -0.625) (layer "F.Fab") (width 0.1))
     (fp_line (start 1 0.625) (end -1 0.625) (layer "F.Fab") (width 0.1))
     (fp_line (start 1 -0.625) (end 1 0.625) (layer "F.Fab") (width 0.1))
@@
     (fp_line (start -1.7 -0.98) (end 1.7 -0.98) (layer "F.CrtYd") (width 0.05))
     (fp_line (start 1.7 0.98) (end -1.7 0.98) (layer "F.CrtYd") (width 0.05))
+    (fp_line (start 1 0.625) (end -1 0.625) (layer "F.Fab") (width 0.1))
     (fp_line (start 1 -0.625) (end 1 0.625) (layer "F.Fab") (width 0.1))
     (fp_line (start -1 0.625) (end -1 -0.625) (layer "F.Fab") (width 0.1))
-    (fp_line (start 1 0.625) (end -1 0.625) (layer "F.Fab") (width 0.1))
     (fp_line (start -1 -0.625) (end 1 -0.625) (layer "F.Fab") (width 0.1))
     (pad "1" smd roundrect locked (at -0.95 0) (size 1 1.45) (layers "F.Cu" "F.Paste" "F.Mask") (roundrect_rratio 0.25)
@@
     (fp_line (start 0 5.15) (end 3.15 5.15) (layer "F.CrtYd") (width 0.05))
     (fp_line (start 0 -5.15) (end -3.15 -5.15) (layer "F.CrtYd") (width 0.05))
+    (fp_line (start 3.75 -3.15) (end 5.15 -3.15) (layer "F.CrtYd") (width 0.05))
     (fp_line (start 5.15 3.15) (end 5.15 0) (layer "F.CrtYd") (width 0.05))
     (fp_line (start 3.75 -3.75) (end 3.75 -3.15) (layer "F.CrtYd") (width 0.05))
@@
     (fp_line (start 3.15 3.75) (end 3.75 3.75) (layer "F.CrtYd") (width 0.05))
     (fp_line (start -3.15 3.75) (end -3.75 3.75) (layer "F.CrtYd") (width 0.05))
-    (fp_line (start 3.75 -3.15) (end 5.15 -3.15) (layer "F.CrtYd") (width 0.05))
     (fp_line (start -2.5 -3.5) (end 3.5 -3.5) (layer "F.Fab") (width 0.1))
     (fp_line (start 3.5 3.5) (end -3.5 3.5) (layer "F.Fab") (width 0.1))
@@
   )
   (footprint "Diode_SMD:D_SOD-123" (layer "B.Cu")
-    (at 52.578 54.356 90)
+    (at 45.301 43.921 180)
     (descr "SOD-123")
     (tags "SOD-123")
@@
     (property "Sheetname" "")
     (attr smd)
-    (fp_text reference "D1" (at 0 2 90) (layer "B.SilkS")
+    (fp_text reference "D1" (at 0 2) (layer "B.SilkS")
       (effects (font (size 1 1) (thickness 0.15)) (justify mirror))
     )
-    (fp_text value "SOD-123" (at 0 -2.1 90) (layer "B.Fab")
+    (fp_text value "SOD-123" (at 0 -2.1) (layer "B.Fab")
       (effects (font (size 1 1) (thickness 0.15)) (justify mirror))
     )
-    (fp_text user "${REFERENCE}" (at 0 2 90) (layer "B.Fab")
+    (fp_text user "${REFERENCE}" (at 0 2) (layer "B.Fab")
       (effects (font (size 1 1) (thickness 0.15)) (justify mirror))
     )
@@
     (fp_line (start -1.4 0.9) (end 1.4 0.9) (layer "B.Fab") (width 0.1))
     (fp_line (start 0.25 0.4) (end 0.25 -0.4) (layer "B.Fab") (width 0.1))
-    (pad "1" smd rect locked (at -1.65 0 90) (size 0.9 1.2) (layers "B.Cu" "B.Paste" "B.Mask")
+    (pad "1" smd rect locked (at -1.65 0 180) (size 0.9 1.2) (layers "B.Cu" "B.Paste" "B.Mask")
       (net 101 "ROW0") (pinfunction "K") (pintype "passive"))
-    (pad "2" smd rect locked (at 1.65 0 90) (size 0.9 1.2) (layers "B.Cu" "B.Paste" "B.Mask")
+    (pad "2" smd rect locked (at 1.65 0 180) (size 0.9 1.2) (layers "B.Cu" "B.Paste" "B.Mask")
       (net 1 "Net-(D1-Pad2)") (pinfunction "A") (pintype "passive"))
     (model "${KICAD6_3DMODEL_DIR}/Diode_SMD.3dshapes/D_SOD-123.wrl"
